File: CC_CV_buck.kicad_pcb (KiCad board)
At the start: 4 copper layers, 115.9 x 39 mm, 78 parts, among them J5 Conn_01x02_Pin, J6 Conn_01x02_Pin, J7 Conn_01x02_Pin, J8 Conn_01x02_Pin, Q1 TIP42C, Q2 AO3400A, Q3 MMBT3906, U1 OPA2197xD, U2 INA194, U3 AOZ6605PI-1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

Commit message: finish stiching and DRC check
Routing:
- net GND: track 11.9 -> 13.2 mm, vias 180 -> 348
